Commit message: finally moves

File: src/Gazebo_world/urdf/robot.xacro (robot description, xacro)
@@ -1,48 +1,7 @@
 <?xml version="1.0"?>
-<robot name="forklift" xmlns:xacro="http://www.ros.org/wiki/xacro">
+<robot name="forklift">
   <!-- Constants -->
-  <xacro:property name="PI" value="3.141592653589793" />
-  <!-- Macro for wheels to avoid repetition -->
-  <xacro:macro name="wheel" params="name parent xyz rpy">
-    <link name="${name}_link">
-      <inertial>
-        <mass value="0.816749" />
-        <origin xyz="-2.21045e-15 -2.33218e-16 -0.0703848" />
-        <inertia ixx="0.0011595" ixy="0" ixz="0"
-                 iyy="0.0011595" iyz="0" izz="0.00147113" />
-      </inertial>
-      <visual>
-        <origin xyz="0 0 -0.1025" rpy="-1.5708 0 0" />
-        <geometry>
-          <mesh filename="file://$(find Gazebo_world)/meshes/wheel1.stl" />
-        </geometry>
-        <material name="wheel_color">
-          <color rgba="0.647059 0.647059 0.647059 1" />
-        </material>
-      </visual>
-      <collision>
-        <origin xyz="0 0 -0.1025" rpy="-1.5708 0 0" />
-        <geometry>
-          <mesh filename="file://$(find Gazebo_world)/meshes/wheel1.stl" />
-        </geometry>
-      </collision>
-    </link>
-    <joint name="${name}" type="revolute">
-      <parent link="${parent}"/>
-      <child link="${name}_link"/>
-      <origin xyz="${xyz}" rpy="${rpy}" />
-      <axis xyz="0 0 1" />
-      <limit effort="10" velocity="10" lower="-${PI}" upper="${PI}" />
-      <dynamics friction="0.0" damping="0.0" />
-    </joint>
-    <!-- Gazebo properties for this wheel -->
-    <gazebo reference="${name}_link">
-      <material>Gazebo/Black</material>
-      <mu1>1.0</mu1>
-      <mu2>1.0</mu2>
-      <kp>1000000.0</kp>
-      <kd>100.0</kd>
-    </gazebo>
-  </xacro:macro>
+  <property name="PI" value="3.141592653589793" />
+  <property name="wheel_radius" value="0.1025" />
   <!-- Base link -->
   <link name="base_link">
@@ -186,15 +145,202 @@
     <parent link="fork" />
     <child link="camera_link" />
-    <origin xyz="0.0 0.0 0.4" rpy="0 0 0" />
-  </joint>
-  <!-- Wheels -->
-  <xacro:wheel name="leftFrontWheel" parent="body"
-               xyz="0.192004 0.25 0.05" rpy="1.5708 0 0" />
-  <xacro:wheel name="leftBackWheel" parent="body"
-               xyz="-0.207996 0.25 0.05" rpy="1.5708 0 0" />
-  <xacro:wheel name="rightFrontWheel" parent="body"
-               xyz="0.192004 -0.25 0.05" rpy="-1.5708 0 0" />
-  <xacro:wheel name="rightBackWheel" parent="body"
-               xyz="-0.207996 -0.25 0.05" rpy="-1.5708 0 0" />
+    <origin xyz="0.0 0.0 0.0" rpy="-3.14 0 0" />
+  </joint>
+  <!-- Left Front Wheel - INDEPENDENT DECLARATION -->
+  <link name="leftFrontWheel_link">
+    <inertial>
+      <mass value="0.816749" />
+      <origin xyz="-2.21045e-15 -2.33218e-16 -0.0703848" />
+      <inertia ixx="0.0011595" ixy="0" ixz="0"
+               iyy="0.0011595" iyz="0" izz="0.00147113" />
+    </inertial>
+    <visual>
+      <origin xyz="0 0 -0.1025" rpy="-1.5708 0 0" />
+      <geometry>
+        <mesh filename="file://$(find Gazebo_world)/meshes/wheel1.stl" />
+      </geometry>
+      <material name="wheel_color">
+        <color rgba="0.647059 0.647059 0.647059 1" />
+      </material>
+    </visual>
+    <collision>
+      <origin xyz="0 0 -0.1025" rpy="-1.5708 0 0" />
+      <geometry>
+        <mesh filename="file://$(find Gazebo_world)/meshes/wheel1.stl" />
+      </geometry>
+    </collision>
+  </link>
+  <joint name="leftFrontWheel" type="continuous">
+    <parent link="body"/>
+    <child link="leftFrontWheel_link"/>
+    <origin xyz="0.192004 0.25 0.05" rpy="1.5708 0 0" />
+    <axis xyz="0 0 -1" />
+    <limit effort="1000" velocity="10"/>
+    <dynamics friction="0.0" damping="0.0" />
+  </joint>
+  <gazebo reference="leftFrontWheel_link">
+    <material>Gazebo/Black</material>
+    <mu1>0.8</mu1>
+    <mu2>0.8</mu2>
+    <kp>1000000.0</kp>
+    <kd>100.0</kd>
+    <surface>
+      <friction>
+        <ode>
+          <mu>0.8</mu>
+          <mu2>0.8</mu2>
+          <slip1>1.0</slip1>
+          <slip2>1.0</slip2>
+        </ode>
+      </friction>
+    </surface>
+  </gazebo>
+  <!-- Left Back Wheel - INDEPENDENT DECLARATION -->
+  <link name="leftBackWheel_link">
+    <inertial>
+      <mass value="0.816749" />
+      <origin xyz="-2.21045e-15 -2.33218e-16 -0.0703848" />
+      <inertia ixx="0.0011595" ixy="0" ixz="0"
+               iyy="0.0011595" iyz="0" izz="0.00147113" />
+    </inertial>
+    <visual>
+      <origin xyz="0 0 -0.1025" rpy="-1.5708 0 0" />
+      <geometry>
+        <mesh filename="file://$(find Gazebo_world)/meshes/wheel1.stl" />
+      </geometry>
+      <material name="wheel_color">
+        <color rgba="0.647059 0.647059 0.647059 1" />
+      </material>
+    </visual>
+    <collision>
+      <origin xyz="0 0 -0.1025" rpy="-1.5708 0 0" />
+      <geometry>
+        <mesh filename="file://$(find Gazebo_world)/meshes/wheel1.stl" />
+      </geometry>
+    </collision>
+  </link>
+  <joint name="leftBackWheel" type="continuous">
+    <parent link="body"/>
+    <child link="leftBackWheel_link"/>
+    <origin xyz="-0.207996 0.25 0.05" rpy="1.5708 0 0" />
+    <axis xyz="0 0 -1" />
+    <limit effort="1000" velocity="10"/>
+    <dynamics friction="0.0" damping="0.0" />
+  </joint>
+  <gazebo reference="leftBackWheel_link">
+    <material>Gazebo/Black</material>
+    <mu1>0.8</mu1>
+    <mu2>0.8</mu2>
+    <kp>1000000.0</kp>
+    <kd>100.0</kd>
+    <surface>
+      <friction>
+        <ode>
+          <mu>0.8</mu>
+          <mu2>0.8</mu2>
+          <slip1>1.0</slip1>
+          <slip2>1.0</slip2>
+        </ode>
+      </friction>
+    </surface>
+  </gazebo>
+  <!-- Right Front Wheel - INDEPENDENT DECLARATION -->
+  <link name="rightFrontWheel_link">
+    <inertial>
+      <mass value="0.816749" />
+      <origin xyz="-2.21045e-15 -2.33218e-16 -0.0703848" />
+      <inertia ixx="0.0011595" ixy="0" ixz="0"
+               iyy="0.0011595" iyz="0" izz="0.00147113" />
+    </inertial>
+    <visual>
+      <origin xyz="0 0 -0.1025" rpy="-1.5708 0 0" />
+      <geometry>
+        <mesh filename="file://$(find Gazebo_world)/meshes/wheel1.stl" />
+      </geometry>
+      <material name="wheel_color">
+        <color rgba="0.647059 0.647059 0.647059 1" />
+      </material>
+    </visual>
+    <collision>
+      <origin xyz="0 0 -0.1025" rpy="-1.5708 0 0" />
+      <geometry>
+        <mesh filename="file://$(find Gazebo_world)/meshes/wheel1.stl" />
+      </geometry>
+    </collision>
+  </link>
+  <joint name="rightFrontWheel" type="continuous">
+    <parent link="body"/>
+    <child link="rightFrontWheel_link"/>
+    <origin xyz="0.192004 -0.25 0.05" rpy="-1.5708 0 0" />
+    <axis xyz="0 0 1" />
+    <limit effort="1000" velocity="10"/>
+    <dynamics friction="0.0" damping="0.0" />
+  </joint>
+  <gazebo reference="rightFrontWheel_link">
+    <material>Gazebo/Black</material>
+    <mu1>0.8</mu1>
+    <mu2>0.8</mu2>
+    <kp>1000000.0</kp>
+    <kd>100.0</kd>
+    <surface>
+      <friction>
+        <ode>
+          <mu>0.8</mu>
+          <mu2>0.8</mu2>
+          <slip1>1.0</slip1>
+          <slip2>1.0</slip2>
+        </ode>
+      </friction>
+    </surface>
+  </gazebo>
+  <!-- Right Back Wheel - INDEPENDENT DECLARATION -->
+  <link name="rightBackWheel_link">
+    <inertial>
+      <mass value="0.816749" />
+      <origin xyz="-2.21045e-15 -2.33218e-16 -0.0703848" />
+      <inertia ixx="0.0011595" ixy="0" ixz="0"
+               iyy="0.0011595" iyz="0" izz="0.00147113" />
+    </inertial>
+    <visual>
+      <origin xyz="0 0 -0.1025" rpy="-1.5708 0 0" />
+      <geometry>
+        <mesh filename="file://$(find Gazebo_world)/meshes/wheel1.stl" />
+      </geometry>
+      <material name="wheel_color">
+        <color rgba="0.647059 0.647059 0.647059 1" />
+      </material>
+    </visual>
+    <collision>
+      <origin xyz="0 0 -0.1025" rpy="-1.5708 0 0" />
+      <geometry>
+        <mesh filename="file://$(find Gazebo_world)/meshes/wheel1.stl" />
+      </geometry>
+    </collision>
+  </link>
+  <joint name="rightBackWheel" type="continuous">
+    <parent link="body"/>
+    <child link="rightBackWheel_link"/>
+    <origin xyz="-0.207996 -0.25 0.05" rpy="-1.5708 0 0" />
+    <axis xyz="0 0 1" />
+    <limit effort="1000" velocity="10"/>
+    <dynamics friction="0.0" damping="0.0" />
+  </joint>
+  <gazebo reference="rightBackWheel_link">
+    <material>Gazebo/Black</material>
+    <mu1>0.8</mu1>
+    <mu2>0.8</mu2>
+    <kp>1000000.0</kp>
+    <kd>100.0</kd>
+    <surface>
+      <friction>
+        <ode>
+          <mu>0.8</mu>
+          <mu2>0.8</mu2>
+          <slip1>1.0</slip1>
+          <slip2>1.0</slip2>
+        </ode>
+      </friction>
+    </surface>
+  </gazebo>
   <!-- Sensors and plugins (these go at the bottom of the file) -->
   <gazebo reference="gps_link">
@@ -235,7 +381,4 @@
           <noise>
             <type>gaussian</type>
-            <!-- Noise is sampled independently per pixel on each frame.
-                  That pixel's noise value is added to each of its color
-                  channels, which at that point lie in the range [0,1]. -->
             <mean>0.0</mean>
             <stddev>0.007</stddev>
@@ -274,29 +417,30 @@
       </sensor>
   </gazebo>
-  <!-- Velocity Control Plugin -->
+  <!-- Velocity Control Plugin - FIXED: SWAPPED LEFT/RIGHT WHEELS -->
 <gazebo>
   <plugin filename="gz-sim-diff-drive-system" name="gz::sim::systems::DiffDrive">
-    <!-- Left wheels (multiple) -->
-    <!-- <left_joint>leftFrontWheel</left_joint> -->
+    <!-- Right wheels become LEFT (to fix rotation direction) -->
+    <left_joint>leftFrontWheel</left_joint>
     <left_joint>leftBackWheel</left_joint>
-    <!-- Right wheels (multiple) -->
-    <!-- <right_joint>rightFrontWheel</right_joint> -->
+    <!-- Left wheels become RIGHT (to fix rotation direction) -->
+    <right_joint>rightFrontWheel</right_joint>
     <right_joint>rightBackWheel</right_joint>
     <!-- Kinematic parameters -->
-    <wheel_separation>0.5</wheel_separation>  <!-- Distance between left and right wheels -->
-    <wheel_radius>0.1025</wheel_radius>        <!-- Radius of your wheels -->
-    <!-- Command and odometry topics -->
+    <wheel_separation>0.5</wheel_separation>
+    <wheel_radius>0.1025</wheel_radius>
+    <!-- Topics -->
     <topic>cmd_vel</topic>
     <odom_topic>odom</odom_topic>
-    <!-- Frame IDs -->
+    <!-- Frames -->
     <frame_id>odom</frame_id>
-    <child_frame_id>base_link</child_frame_id>  <!-- Must match your URDF root -->
-    <!-- Publishing rates -->
+    <child_frame_id>base_link</child_frame_id>
     <odom_publisher_frequency>30.0</odom_publisher_frequency>
-    <!-- TF publication -->
-    <tf_topic>/tf</tf_topic>
-    <publish_tf>true</publish_tf>  <!-- Ensure TF is published -->
+    <publish_tf>true</publish_tf>
+    <!-- Critical additions for better performance -->
+    <max_wheel_torque>500</max_wheel_torque>
+    <max_wheel_acceleration>5</max_wheel_acceleration>
   </plugin>
 </gazebo>
+  <!-- Joint State Publisher -->
   <gazebo>
     <plugin filename="gz-sim-joint-state-publisher-system" name="gz::sim::systems::JointStatePublisher">
@@ -311,8 +455,12 @@
       <joint_name>lift</joint_name>
     </plugin>
-    <plugin filename="gz-sim-sensors-system"
-            name="gz::sim::systems::Sensors">
+    <plugin filename="gz-sim-sensors-system" name="gz::sim::systems::Sensors">
       <render_engine>ogre2</render_engine>
     </plugin>
+    <!-- Joint Controller -->
+    <plugin filename="gz-sim-joint-controller-system" name="gz::sim::systems::JointController">
+      <joint_name>lift</joint_name>
+      <initial_velocity>1.0</initial_velocity>
+    </plugin>
   </gazebo>
 </robot>
